File: Hardware/SparkFun_Beefcake_Relay_Control_Kit.brd (EAGLE design)
At the start: 62.2 x 30.5 mm, 18 parts, among them K1 JQX-15F, Q2 2N3904

Commit message: Resolved github issues
Parts:
- renumbered Q2 to Q1, R4 to R3
Changed lines of the file:
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@@
 <layer number="21" name="tPlace" color="16" fill="1" visible="yes" active="yes"/>
 <layer number="22" name="bPlace" color="14" fill="1" visible="yes" active="yes"/>
-<layer number="23" name="tOrigins" color="15" fill="1" visible="no" active="yes"/>
-<layer number="24" name="bOrigins" color="15" fill="1" visible="no" active="yes"/>
+<layer number="23" name="tOrigins" color="15" fill="1" visible="yes" active="yes"/>
+<layer number="24" name="bOrigins" color="15" fill="1" visible="yes" active="yes"/>
 <layer number="25" name="tNames" color="7" fill="1" visible="no" active="yes"/>
 <layer number="26" name="bNames" color="7" fill="1" visible="no" active="yes"/>
@@
 <layer number="28" name="bValues" color="7" fill="1" visible="no" active="yes"/>
 <layer number="29" name="tStop" color="7" fill="3" visible="no" active="yes"/>
-<layer number="30" name="bStop" color="7" fill="6" visible="yes" active="yes"/>
+<layer number="30" name="bStop" color="7" fill="6" visible="no" active="yes"/>
 <layer number="31" name="tCream" color="7" fill="4" visible="no" active="yes"/>
 <layer number="32" name="bCream" color="7" fill="5" visible="no" active="yes"/>
@@
 <layer number="43" name="vRestrict" color="2" fill="10" visible="no" active="yes"/>
 <layer number="44" name="Drills" color="7" fill="1" visible="no" active="yes"/>
-<layer number="45" name="Holes" color="7" fill="1" visible="no" active="yes"/>
+<layer number="45" name="Holes" color="7" fill="1" visible="yes" active="yes"/>
 <layer number="46" name="Milling" color="3" fill="1" visible="no" active="yes"/>
 <layer number="47" name="Measures" color="7" fill="1" visible="no" active="yes"/>
@@
 </autorouter>
 <elements>
-<element name="Q2" library="SparkFun-DiscreteSemi" package="TO-92-EZ" value="2N3904" x="48.26" y="10.4775" smashed="yes" rot="R270">
+<element name="Q1" library="SparkFun-DiscreteSemi" package="TO-92-EZ" value="2N3904" x="48.26" y="10.4775" smashed="yes" rot="R270">
 <attribute name="NAME" x="46.99" y="14.9225" size="0.8128" layer="25" font="vector" ratio="15" align="center"/>
 <attribute name="VALUE" x="48.5775" y="13.97" size="0.8128" layer="27" font="vector" ratio="15" align="center"/>
@@
 <attribute name="PROD_ID" value="DIO-09529" x="49.8475" y="18.7325" size="1.778" layer="27" rot="R90" display="off"/>
 </element>
-<element name="R4" library="SparkFun-Resistors" package="AXIAL-0.3EZ" value="1K" x="51.1175" y="23.1775" smashed="yes">
+<element name="R3" library="SparkFun-Resistors" package="AXIAL-0.3EZ" value="1K" x="51.1175" y="23.1775" smashed="yes">
 <attribute name="VALUE" value="1K" x="51.1175" y="23.1775" size="1.778" layer="27" display="off"/>
 <attribute name="PROD_ID" value="RES-12182" x="51.1175" y="23.1775" size="1.778" layer="27" display="off"/>
@@
 <element name="JP1" library="SparkFun-Passives" package="PAD-JUMPER-2-NO_YES_SILK" value="JUMPER-PAD-2-NOYES_SILK" x="47.9425" y="3.4925" rot="MR180"/>
 <element name="D2" library="SparkFun-DiscreteSemi" package="DIODE-1N4148-KIT" value="Zener" x="47.9425" y="3.4925" smashed="yes" rot="R180">
-<attribute name="PROD_ID" value="Generic" x="47.9425" y="3.4925" size="1.778" layer="27" rot="R180" display="off"/>
+<attribute name="PROD_ID" value="DIO-13313" x="47.9425" y="3.4925" size="1.778" layer="27" rot="R180" display="off"/>
 <attribute name="NAME" x="50.4825" y="2.2225" size="0.4064" layer="25" rot="R180"/>
-<attribute name="VALUE" x="49.9745" y="4.0005" size="0.8128" layer="21" font="vector" ratio="15" rot="R180"/>
+<attribute name="VALUE" value="Zener" x="46.2915" y="3.4925" size="0.8128" layer="21" font="vector" ratio="15" align="center-left"/>
 </element>
 </elements>
 <signals>
 <signal name="GND">
-<contactref element="Q2" pad="1"/>
+<contactref element="Q1" pad="1"/>
 <contactref element="J2" pad="1"/>
 <wire x1="48.26" y1="11.7475" x2="49.2125" y2="12.7" width="0.6096" layer="1"/>
@@
 </signal>
 <signal name="N$6">
-<contactref element="Q2" pad="2"/>
+<contactref element="Q1" pad="2"/>
 <contactref element="R2" pad="P$1"/>
 <wire x1="50.165" y1="10.4775" x2="50.165" y2="6.985" width="0.6096" layer="1"/>
@@
 <signal name="N$9">
 <contactref element="LED1" pad="K"/>
-<contactref element="R4" pad="P$2"/>
+<contactref element="R3" pad="P$2"/>
 <wire x1="49.8475" y1="20.0025" x2="53.34" y2="20.0025" width="0.6096" layer="1"/>
 <wire x1="53.34" y1="20.0025" x2="54.9275" y2="21.59" width="0.6096" layer="1"/>
@@
 </signal>
 <signal name="COIL">
-<contactref element="Q2" pad="3"/>
-<contactref element="R4" pad="P$1"/>
+<contactref element="Q1" pad="3"/>
+<contactref element="R3" pad="P$1"/>
 <contactref element="K1" pad="COIL2"/>
 <wire x1="48.26" y1="9.2075" x2="48.26" y2="6.985" width="0.6096" layer="1"/>
