File: Hardware/SparkFun_Beefcake_Relay_Control_Kit.sch (EAGLE design)
At the start: 16 parts, among them Q2 2N3904, U6 RELAYPTH3

Commit message: Design ready for proto 1 review
Parts:
- removed JP3: Load, SparkFun:M025MM
- removed R1: 10K, SparkFun:RESISTORAXIAL-0.3
- removed U$1: LOGO-SFENEW, SparkFun:LOGO-SFENEW
- added D2: BZT52, SparkFun-DiscreteSemi:DIODE-ZENER
- added JP1: (no value), SparkFun-Connectors:M03-SCREW-5MM
- added LOGO1: SFE_LOGO_NAME_FLAME.2_INCH, SparkFun-Aesthetics:SFE_LOGO_NAME_FLAME.2_INCH
- D1: device SparkFun:DIODE1N4148 -> SparkFun-DiscreteSemi:DIODE1N4148
- JP2: device SparkFun:M03SCREW -> SparkFun-Connectors:M03SCREW
- LED1: device SparkFun:LED5MM -> SparkFun-LED:LED5MM
- Q2: device SparkFun:TRANSISTOR_NPNTO92 -> SparkFun-DiscreteSemi:TRANSISTOR_NPN2N3904
- R2, R4: device SparkFun:RESISTORAXIAL-0.3 -> SparkFun-Resistors:1KOHM-1/4W-5%(PTH)
- U6: value RELAYPTH3 -> JQX-15F; device SparkFun:RELAYPTH3 -> SparkFun-Electromechanical:RELAYPTH5
- renumbered FRAME1 to FRAME2
Connections:
- removed net LOAD1: JP3.2, U6.MAIN
- removed net LOAD2: JP3.1, U6.NO
- new net COMMON: JP1.3, U6.MAIN
- new net NC: JP1.1, U6.NC
- new net NO: JP1.2, U6.NO
- net COIL: now also D2.A, D2.C
- net GND: no longer R1.2
- net N$6: no longer R1.1
Other:
- note added: "CAUTION!"
- note added: "Flyback Arrestor -- Place D1 with a normal diode such as the 1N4148 for normal use. For low voltage cutout, use a zener at D2 and cut the bypass trace."
- note added: "If metal standoffs are required, or mounting to a conductive chassis, standoff diameter must be less than 0.21 inch."
- note added: "N. Seidle, M Taylor, SparkFun Electronics"
- note added: "Relay drive indicator -- Illuminates when the relay coil is energized"
- note added: "To maintiain 250VAC/VDC galvanic isolation, use non-conductive standoffs and 4-40 HW with a head diameter no greater than 0.21 inch."
- note added: "v18"
- note removed: "17"
- note removed: "N. Seidle, SparkFun Electronics"
- moved on the sheet: JP2, Q2, R2, R4, U6

Commit message: Running through review changes
Parts:
- added JP3: JUMPER-PAD-2-NC_BY_TRACE, SparkFun-Passives:JUMPER-PAD-2-NC_BY_TRACE
- D1: device SparkFun-DiscreteSemi:DIODE1N4148 -> SparkFun-DiscreteSemi:DIODEKIT
- D2: device SparkFun-DiscreteSemi:DIODE-ZENER -> SparkFun-DiscreteSemi:DIODEKIT
- LED1: device SparkFun-LED:LED5MM -> SparkFun-LED:LED5MM-KIT
- LOGO1: value SFE_LOGO_NAME_FLAME.2_INCH -> SFE_LOGO_NAME_FLAME.1_INCH; device SparkFun-Aesthetics:SFE_LOGO_NAME_FLAME.2_INCH -> SparkFun-Aesthetics:SFE_LOGO_NAME_FLAME.1_INCH
- Q2: device SparkFun-DiscreteSemi:TRANSISTOR_NPN2N3904 -> SparkFun-DiscreteSemi:TRANSISTOR_NPN2N3904-EZ
- R2, R4: value 1K -> 1k; device SparkFun-Resistors:1KOHM-1/4W-5%(PTH) -> SparkFun-Resistors:RESISTOREZ
Connections:
- net COIL: now also JP3.1, JP3.2
Changed lines of the file:
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@@
 </classes>
 <parts>
-<part name="Q2" library="SparkFun-DiscreteSemi" deviceset="TRANSISTOR_NPN" device="2N3904" value="2N3904"/>
+<part name="Q2" library="SparkFun-DiscreteSemi" deviceset="TRANSISTOR_NPN" device="2N3904-EZ" value="2N3904"/>
 <part name="GND1" library="SparkFun" deviceset="GND" device=""/>
 <part name="U$2" library="SparkFun" deviceset="RAW" device=""/>
-<part name="R2" library="SparkFun-Resistors" deviceset="1KOHM-1/4W-5%(PTH)" device="" value="1K"/>
-<part name="LED1" library="SparkFun-LED" deviceset="LED" device="5MM"/>
-<part name="R4" library="SparkFun-Resistors" deviceset="1KOHM-1/4W-5%(PTH)" device="" value="1K"/>
+<part name="R2" library="SparkFun-Resistors" deviceset="RESISTOR" device="EZ" value="1k"/>
+<part name="LED1" library="SparkFun-LED" deviceset="LED" device="5MM-KIT"/>
+<part name="R4" library="SparkFun-Resistors" deviceset="RESISTOR" device="EZ" value="1k"/>
 <part name="U$3" library="SparkFun" deviceset="STAND-OFF" device=""/>
 <part name="U$4" library="SparkFun" deviceset="STAND-OFF" device=""/>
 <part name="U$5" library="SparkFun" deviceset="STAND-OFF" device=""/>
 <part name="U$7" library="SparkFun" deviceset="STAND-OFF" device=""/>
-<part name="D1" library="SparkFun-DiscreteSemi" deviceset="DIODE" device="1N4148" value="1N4148"/>
+<part name="D1" library="SparkFun-DiscreteSemi" deviceset="DIODE" device="KIT" value="1N4148"/>
 <part name="U$10" library="SparkFun" deviceset="RAW" device=""/>
 <part name="GND2" library="SparkFun" deviceset="GND" device=""/>
@@
 <part name="U$12" library="SparkFun" deviceset="OSHW-LOGO" device="S"/>
 <part name="JP1" library="SparkFun-Connectors" deviceset="M03" device="-SCREW-5MM"/>
-<part name="D2" library="SparkFun-DiscreteSemi" deviceset="DIODE-ZENER" device="" value="BZT52"/>
+<part name="D2" library="SparkFun-DiscreteSemi" deviceset="DIODE" device="KIT" value="BZT52"/>
 <part name="FRAME2" library="SparkFun-Aesthetics" deviceset="FRAME-LETTER" device=""/>
-<part name="LOGO1" library="SparkFun-Aesthetics" deviceset="SFE_LOGO_NAME_FLAME" device=".2_INCH" value="SFE_LOGO_NAME_FLAME.2_INCH"/>
+<part name="LOGO1" library="SparkFun-Aesthetics" deviceset="SFE_LOGO_NAME_FLAME" device=".1_INCH" value="SFE_LOGO_NAME_FLAME.1_INCH"/>
+<part name="JP3" library="SparkFun-Passives" deviceset="JUMPER-PAD-2-NC_BY_TRACE" device=""/>
 </parts>
 <sheets>
@@
 <instance part="D1" gate="G$1" x="106.68" y="147.32" smashed="yes" rot="R90">
 <attribute name="NAME" x="109.474" y="146.304" size="1.778" layer="95"/>
-<attribute name="VALUE" x="109.474" y="144.018" size="1.778" layer="96"/>
 </instance>
 <instance part="U$10" gate="G$1" x="134.62" y="93.98"/>
@@
 <instance part="D2" gate="G$1" x="106.68" y="132.08" smashed="yes" rot="R270">
 <attribute name="NAME" x="109.22" y="131.2926" size="1.778" layer="95"/>
-<attribute name="VALUE" x="109.22" y="129.0066" size="1.778" layer="96"/>
 </instance>
 <instance part="FRAME2" gate="G$1" x="0" y="0"/>
 <instance part="FRAME2" gate="V" x="147.32" y="0"/>
 <instance part="LOGO1" gate="G$1" x="149.86" y="43.18"/>
+<instance part="JP3" gate="G$1" x="99.06" y="132.08" rot="R90"/>
 </instances>
 <busses>
@@
 <wire x1="106.68" y1="119.38" x2="129.54" y2="119.38" width="0.1524" layer="91"/>
 <pinref part="D2" gate="G$1" pin="C"/>
-<wire x1="106.68" y1="129.54" x2="106.68" y2="127" width="0.1524" layer="91"/>
-<wire x1="106.68" y1="119.38" x2="106.68" y2="127" width="0.1524" layer="91"/>
-<wire x1="106.68" y1="127" x2="99.06" y2="127" width="0.1524" layer="91"/>
+<wire x1="106.68" y1="129.54" x2="106.68" y2="124.46" width="0.1524" layer="91"/>
+<wire x1="106.68" y1="119.38" x2="106.68" y2="124.46" width="0.1524" layer="91"/>
+<wire x1="106.68" y1="124.46" x2="99.06" y2="124.46" width="0.1524" layer="91"/>
+<junction x="106.68" y="124.46"/>
+<junction x="106.68" y="119.38"/>
+<junction x="106.68" y="68.58"/>
+<pinref part="JP3" gate="G$1" pin="1"/>
+<wire x1="99.06" y1="127" x2="99.06" y2="124.46" width="0.2032" layer="91"/>
+</segment>
+<segment>
+<pinref part="JP3" gate="G$1" pin="2"/>
 <pinref part="D1" gate="G$1" pin="A"/>
+<wire x1="106.68" y1="144.78" x2="106.68" y2="139.7" width="0.1524" layer="91"/>
 <pinref part="D2" gate="G$1" pin="A"/>
-<wire x1="106.68" y1="144.78" x2="106.68" y2="137.16" width="0.1524" layer="91"/>
-<wire x1="106.68" y1="134.62" x2="106.68" y2="137.16" width="0.1524" layer="91"/>
-<wire x1="106.68" y1="137.16" x2="99.06" y2="137.16" width="0.1524" layer="91"/>
-<wire x1="99.06" y1="137.16" x2="99.06" y2="127" width="0.1524" layer="91"/>
-<junction x="106.68" y="127"/>
-<junction x="106.68" y="119.38"/>
-<junction x="106.68" y="137.16"/>
-<junction x="106.68" y="68.58"/>
+<wire x1="106.68" y1="134.62" x2="106.68" y2="139.7" width="0.1524" layer="91"/>
+<junction x="106.68" y="139.7"/>
+<wire x1="106.68" y1="139.7" x2="99.06" y2="139.7" width="0.1524" layer="91"/>
+<wire x1="99.06" y1="139.7" x2="99.06" y2="137.16" width="0.2032" layer="91"/>
 </segment>
 </net>

Commit message: Ready for QC's review
Parts:
- D1: PROD_ID (none) -> DIO-08378
- D2: PROD-ID (none) -> DIO-08199
- LED1: PROD_ID (none) -> DIO-09529
- R2, R4: value 1k -> 1K; device SparkFun-Resistors:RESISTOREZ -> SparkFun-Resistors:1KOHM-1/4W-1%(PTH)HORIZ-KIT
Other:
- note added: "Supply RAW with 5v DC"
- note added: "v20"
- note removed: "v18"
Changed lines of the file:
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@@
 <part name="GND1" library="SparkFun" deviceset="GND" device=""/>
 <part name="U$2" library="SparkFun" deviceset="RAW" device=""/>
-<part name="R2" library="SparkFun-Resistors" deviceset="RESISTOR" device="EZ" value="1k"/>
-<part name="LED1" library="SparkFun-LED" deviceset="LED" device="5MM-KIT"/>
-<part name="R4" library="SparkFun-Resistors" deviceset="RESISTOR" device="EZ" value="1k"/>
+<part name="R2" library="SparkFun-Resistors" deviceset="1KOHM-1/4W-1%(PTH)" device="HORIZ-KIT" value="1K"/>
+<part name="LED1" library="SparkFun-LED" deviceset="LED" device="5MM-KIT">
+<attribute name="PROD_ID" value="DIO-09529"/>
+</part>
+<part name="R4" library="SparkFun-Resistors" deviceset="1KOHM-1/4W-1%(PTH)" device="HORIZ-KIT" value="1K"/>
 <part name="U$3" library="SparkFun" deviceset="STAND-OFF" device=""/>
 <part name="U$4" library="SparkFun" deviceset="STAND-OFF" device=""/>
 <part name="U$5" library="SparkFun" deviceset="STAND-OFF" device=""/>
 <part name="U$7" library="SparkFun" deviceset="STAND-OFF" device=""/>
-<part name="D1" library="SparkFun-DiscreteSemi" deviceset="DIODE" device="KIT" value="1N4148"/>
+<part name="D1" library="SparkFun-DiscreteSemi" deviceset="DIODE" device="KIT" value="1N4148">
+<attribute name="PROD_ID" value="DIO-08378"/>
+</part>
 <part name="U$10" library="SparkFun" deviceset="RAW" device=""/>
 <part name="GND2" library="SparkFun" deviceset="GND" device=""/>
@@
 <part name="U$12" library="SparkFun" deviceset="OSHW-LOGO" device="S"/>
 <part name="JP1" library="SparkFun-Connectors" deviceset="M03" device="-SCREW-5MM"/>
-<part name="D2" library="SparkFun-DiscreteSemi" deviceset="DIODE" device="KIT" value="BZT52"/>
+<part name="D2" library="SparkFun-DiscreteSemi" deviceset="DIODE" device="KIT" value="BZT52">
+<attribute name="PROD-ID" value="DIO-08199"/>
+</part>
 <part name="FRAME2" library="SparkFun-Aesthetics" deviceset="FRAME-LETTER" device=""/>
 <part name="LOGO1" library="SparkFun-Aesthetics" deviceset="SFE_LOGO_NAME_FLAME" device=".1_INCH" value="SFE_LOGO_NAME_FLAME.1_INCH"/>
@@
 <text x="171.704" y="8.89" size="1.778" layer="94">N. Seidle, M Taylor,
 SparkFun Electronics</text>
-<text x="240.284" y="7.112" size="2.54" layer="94">v18</text>
+<text x="240.284" y="7.112" size="2.54" layer="94">v20</text>
 <text x="142.24" y="86.36" size="2.032" layer="97">Relay drive indicator -- Illuminates
 when the relay coil is energized</text>
@@
 conductive chassis, standoff diameter must be less
 than 0.21 inch.</text>
+<text x="63.5" y="68.58" size="2.032" layer="97">Supply RAW with 5v DC</text>
 </plain>
 <instances>
@@
 <instance part="U$2" gate="G$1" x="106.68" y="154.94"/>
 <instance part="R2" gate="G$1" x="91.44" y="53.34" rot="R180"/>
-<instance part="LED1" gate="G$1" x="134.62" y="88.9"/>
+<instance part="LED1" gate="G$1" x="134.62" y="88.9">
+<attribute name="PROD_ID" x="134.62" y="88.9" size="1.27" layer="96" display="both"/>
+</instance>
 <instance part="R4" gate="G$1" x="134.62" y="76.2" rot="R90"/>
 <instance part="U$3" gate="G$1" x="246.38" y="25.4"/>
@@
 <instance part="U$7" gate="G$1" x="231.14" y="25.4"/>
 <instance part="D1" gate="G$1" x="106.68" y="147.32" smashed="yes" rot="R90">
-<attribute name="NAME" x="109.474" y="146.304" size="1.778" layer="95"/>
+<attribute name="PROD_ID" x="106.68" y="147.32" size="1.27" layer="96" rot="R90" display="off"/>
+<attribute name="NAME" x="108.7374" y="142.24" size="1.778" layer="95" rot="R90"/>
+<attribute name="VALUE" x="111.5314" y="142.24" size="1.778" layer="96" rot="R90"/>
 </instance>
 <instance part="U$10" gate="G$1" x="134.62" y="93.98"/>
@@
 <instance part="U$8" gate="G$1" x="81.28" y="58.42"/>
 <instance part="U6" gate="G$1" x="139.7" y="124.46"/>
-<instance part="U$12" gate="G$1" x="132.08" y="12.7"/>
+<instance part="U$12" gate="G$1" x="167.64" y="48.26"/>
 <instance part="JP1" gate="G$1" x="182.88" y="139.7" rot="R180"/>
 <instance part="D2" gate="G$1" x="106.68" y="132.08" smashed="yes" rot="R270">
-<attribute name="NAME" x="109.22" y="131.2926" size="1.778" layer="95"/>
+<attribute name="NAME" x="108.7374" y="127" size="1.778" layer="95" rot="R90"/>
+<attribute name="VALUE" x="111.5314" y="127" size="1.778" layer="96" rot="R90"/>
 </instance>
 <instance part="FRAME2" gate="G$1" x="0" y="0"/>
 <instance part="FRAME2" gate="V" x="147.32" y="0"/>
-<instance part="LOGO1" gate="G$1" x="149.86" y="43.18"/>
-<instance part="JP3" gate="G$1" x="99.06" y="132.08" rot="R90"/>
+<instance part="LOGO1" gate="G$1" x="185.42" y="38.1"/>
+<instance part="JP3" gate="G$1" x="99.06" y="132.08" smashed="yes" rot="R90">
+<attribute name="NAME" x="96.52" y="129.54" size="1.778" layer="95" rot="R90"/>
+</instance>
 </instances>
 <busses>
@@
 </sheet>
 </sheets>
+<errors>
+</errors>
 </schematic>
 </drawing>

Commit message: updated bom
Parts:
- removed JP3: JUMPER-PAD-2-NC_BY_TRACE, SparkFun-Passives:JUMPER-PAD-2-NC_BY_TRACE
- removed U6: JQX-15F, SparkFun-Electromechanical:RELAYPTH5
- added J1: (no value), SparkFun-Connectors:M03-SCREW-5MM
- added K1: JQX-15F, SparkFun-Electromechanical:RELAYPTH5
- JP1: value (none) -> JUMPER-PAD-2-NC_BY_TRACE; device SparkFun-Connectors:M03-SCREW-5MM -> SparkFun-Passives:JUMPER-PAD-2-NC_BY_TRACE
- renumbered JP2 to J2
Connections:
- net COIL: now also JP1.1, JP1.2, K1.COIL2; no longer JP3.1, JP3.2, U6.COIL2
- net COMMON: now also J1.3, K1.MAIN; no longer JP1.3, U6.MAIN
- net NC: now also J1.1, K1.NC; no longer JP1.1, U6.NC
- net NO: now also J1.2, K1.NO; no longer JP1.2, U6.NO
- net RAW: now also K1.COIL1; no longer U6.COIL1
Changed lines of the file:
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@@
 <part name="U$10" library="SparkFun" deviceset="RAW" device=""/>
 <part name="GND2" library="SparkFun" deviceset="GND" device=""/>
-<part name="JP2" library="SparkFun-Connectors" deviceset="M03" device="SCREW"/>
+<part name="J2" library="SparkFun-Connectors" deviceset="M03" device="SCREW"/>
 <part name="U$8" library="SparkFun" deviceset="RAW" device=""/>
-<part name="U6" library="SparkFun-Electromechanical" deviceset="RELAY" device="PTH5" value="JQX-15F"/>
+<part name="K1" library="SparkFun-Electromechanical" deviceset="RELAY" device="PTH5" value="JQX-15F"/>
 <part name="U$12" library="SparkFun" deviceset="OSHW-LOGO" device="S"/>
-<part name="JP1" library="SparkFun-Connectors" deviceset="M03" device="-SCREW-5MM"/>
+<part name="J1" library="SparkFun-Connectors" deviceset="M03" device="-SCREW-5MM">
+<attribute name="PROD_ID" value="CONN-10134"/>
+</part>
 <part name="D2" library="SparkFun-DiscreteSemi" deviceset="DIODE" device="KIT" value="BZT52">
 <attribute name="PROD-ID" value="DIO-08199"/>
@@
 <part name="FRAME2" library="SparkFun-Aesthetics" deviceset="FRAME-LETTER" device=""/>
 <part name="LOGO1" library="SparkFun-Aesthetics" deviceset="SFE_LOGO_NAME_FLAME" device=".1_INCH" value="SFE_LOGO_NAME_FLAME.1_INCH"/>
-<part name="JP3" library="SparkFun-Passives" deviceset="JUMPER-PAD-2-NC_BY_TRACE" device=""/>
+<part name="JP1" library="SparkFun-Passives" deviceset="JUMPER-PAD-2-NC_BY_TRACE" device=""/>
 </parts>
 <sheets>
@@
 <instance part="U$2" gate="G$1" x="106.68" y="154.94"/>
 <instance part="R2" gate="G$1" x="91.44" y="53.34" rot="R180"/>
-<instance part="LED1" gate="G$1" x="134.62" y="88.9">
-<attribute name="PROD_ID" x="134.62" y="88.9" size="1.27" layer="96" display="both"/>
+<instance part="LED1" gate="G$1" x="134.62" y="88.9" smashed="yes">
+<attribute name="NAME" x="138.176" y="84.328" size="1.778" layer="95" rot="R90"/>
+<attribute name="VALUE" x="140.335" y="84.328" size="1.778" layer="96" rot="R90"/>
 </instance>
 <instance part="R4" gate="G$1" x="134.62" y="76.2" rot="R90"/>
@@
 <instance part="U$10" gate="G$1" x="134.62" y="93.98"/>
 <instance part="GND2" gate="1" x="81.28" y="45.72"/>
-<instance part="JP2" gate="G$1" x="66.04" y="53.34"/>
+<instance part="J2" gate="G$1" x="66.04" y="53.34"/>
 <instance part="U$8" gate="G$1" x="81.28" y="58.42"/>
-<instance part="U6" gate="G$1" x="139.7" y="124.46"/>
+<instance part="K1" gate="K$1" x="139.7" y="124.46"/>
 <instance part="U$12" gate="G$1" x="167.64" y="48.26"/>
-<instance part="JP1" gate="G$1" x="182.88" y="139.7" rot="R180"/>
+<instance part="J1" gate="G$1" x="182.88" y="139.7" rot="R180">
+<attribute name="PROD_ID" x="182.88" y="139.7" size="1.27" layer="96" rot="R180" display="off"/>
+</instance>
 <instance part="D2" gate="G$1" x="106.68" y="132.08" smashed="yes" rot="R270">
 <attribute name="NAME" x="108.7374" y="127" size="1.778" layer="95" rot="R90"/>
@@
 <instance part="FRAME2" gate="V" x="147.32" y="0"/>
 <instance part="LOGO1" gate="G$1" x="185.42" y="38.1"/>
-<instance part="JP3" gate="G$1" x="99.06" y="132.08" smashed="yes" rot="R90">
+<instance part="JP1" gate="G$1" x="99.06" y="132.08" smashed="yes" rot="R90">
 <attribute name="NAME" x="96.52" y="129.54" size="1.778" layer="95" rot="R90"/>
 </instance>
@@
 <wire x1="81.28" y1="50.8" x2="81.28" y2="48.26" width="0.1524" layer="91"/>
 <pinref part="GND2" gate="1" pin="GND"/>
-<pinref part="JP2" gate="G$1" pin="1"/>
+<pinref part="J2" gate="G$1" pin="1"/>
 </segment>
 </net>
@@
 <pinref part="U$2" gate="G$1" pin="RAW"/>
 <pinref part="D1" gate="G$1" pin="C"/>
-<pinref part="U6" gate="G$1" pin="COIL1"/>
+<pinref part="K1" gate="K$1" pin="COIL1"/>
 </segment>
 <segment>
@@
 <wire x1="73.66" y1="55.88" x2="81.28" y2="55.88" width="0.1524" layer="91"/>
 <wire x1="81.28" y1="55.88" x2="81.28" y2="58.42" width="0.1524" layer="91"/>
-<pinref part="JP2" gate="G$1" pin="3"/>
+<pinref part="J2" gate="G$1" pin="3"/>
 <pinref part="U$8" gate="G$1" pin="RAW"/>
 </segment>
@@
 <label x="76.708" y="53.594" size="1.778" layer="95"/>
 <pinref part="R2" gate="G$1" pin="2"/>
-<pinref part="JP2" gate="G$1" pin="2"/>
+<pinref part="J2" gate="G$1" pin="2"/>
 </segment>
 </net>
@@
 <wire x1="106.68" y1="58.42" x2="106.68" y2="68.58" width="0.1524" layer="91"/>
 <wire x1="106.68" y1="68.58" x2="106.68" y2="119.38" width="0.1524" layer="91"/>
-<pinref part="U6" gate="G$1" pin="COIL2"/>
+<pinref part="K1" gate="K$1" pin="COIL2"/>
 <wire x1="106.68" y1="119.38" x2="129.54" y2="119.38" width="0.1524" layer="91"/>
 <pinref part="D2" gate="G$1" pin="C"/>
@@
 <junction x="106.68" y="119.38"/>
 <junction x="106.68" y="68.58"/>
-<pinref part="JP3" gate="G$1" pin="1"/>
+<pinref part="JP1" gate="G$1" pin="1"/>
 <wire x1="99.06" y1="127" x2="99.06" y2="124.46" width="0.2032" layer="91"/>
 </segment>
 <segment>
-<pinref part="JP3" gate="G$1" pin="2"/>
+<pinref part="JP1" gate="G$1" pin="2"/>
 <pinref part="D1" gate="G$1" pin="A"/>
 <wire x1="106.68" y1="144.78" x2="106.68" y2="139.7" width="0.1524" layer="91"/>
@@
 <wire x1="167.64" y1="124.46" x2="147.32" y2="124.46" width="0.1524" layer="91"/>
 <label x="149.86" y="124.46" size="1.778" layer="95"/>
-<pinref part="JP1" gate="G$1" pin="3"/>
+<pinref part="J1" gate="G$1" pin="3"/>
 <wire x1="167.64" y1="124.46" x2="167.64" y2="137.16" width="0.1524" layer="91"/>
 <wire x1="167.64" y1="137.16" x2="175.26" y2="137.16" width="0.1524" layer="91"/>
-<pinref part="U6" gate="G$1" pin="MAIN"/>
+<pinref part="K1" gate="K$1" pin="MAIN"/>
 </segment>
 </net>
@@
 <wire x1="165.1" y1="119.38" x2="147.32" y2="119.38" width="0.1524" layer="91"/>
 <label x="152.4" y="119.38" size="1.778" layer="95"/>
-<pinref part="JP1" gate="G$1" pin="2"/>
+<pinref part="J1" gate="G$1" pin="2"/>
 <wire x1="165.1" y1="119.38" x2="165.1" y2="139.7" width="0.1524" layer="91"/>
 <wire x1="165.1" y1="139.7" x2="175.26" y2="139.7" width="0.1524" layer="91"/>
-<pinref part="U6" gate="G$1" pin="NO"/>
+<pinref part="K1" gate="K$1" pin="NO"/>
 </segment>
 </net>
@@
 <wire x1="147.32" y1="129.54" x2="162.56" y2="129.54" width="0.1524" layer="91"/>
 <label x="152.4" y="129.54" size="1.778" layer="95"/>
-<pinref part="JP1" gate="G$1" pin="1"/>
+<pinref part="J1" gate="G$1" pin="1"/>
 <wire x1="162.56" y1="129.54" x2="162.56" y2="142.24" width="0.1524" layer="91"/>
 <wire x1="162.56" y1="142.24" x2="175.26" y2="142.24" width="0.1524" layer="91"/>
-<pinref part="U6" gate="G$1" pin="NC"/>
-</segment>
-</net>
+<pinref part="K1" gate="K$1" pin="NC"/>
+</segment>
+</net>
